File: itx4ups_pro_pcb/itx4ups_pro_pcb/itx4ups_pro_pcb.kicad_sch (KiCad schematic)
At the start: 20 parts, among them J1 ATX-24

Commit message: pcb added
Signed-off-by: xianii <jiyucheng007@gmail.com>
Parts:
- removed H8: UpBoard_Hole, symbol Mechanical:MountingHole
- removed J? (x2): USB_A, symbol Connector:USB_A
- added H10, H11, H9: Rpi_ZeroW2_Hole, MountingHole:MountingHole_3.2mm_M3_ISO14580_Pad, symbol Mechanical:MountingHole
- added H12, H13, H14, H15: RPI4_Hole, MountingHole:MountingHole_3.2mm_M3_ISO14580_Pad, symbol Mechanical:MountingHole
- added J10: Conn_01x02, Connector_PinHeader_2.54mm:PinHeader_1x02_P2.54mm_Vertical, symbol Connector_Generic:Conn_01x02
- added J11, J18, J19: Conn_01x04, Connector_TE-Connectivity:TE_MATE-N-LOK_350211-1_1x04_P5.08mm_Vertical, symbol Connector_Generic:Conn_01x04
- added J12: Conn_01x02, LED_THT:LED_D3.0mm, symbol Connector_Generic:Conn_01x02
- added J15: Conn_01x08, Library:USB-double, symbol Connector_Generic:Conn_01x08
- added J17: Conn_01x02, Library:PWR_Switch_Pad, symbol Connector_Generic:Conn_01x02
- added J4: Conn_01x04, Connector_PinHeader_2.54mm:PinHeader_1x04_P2.54mm_Vertical, symbol Connector_Generic:Conn_01x04
- added J9: Jack-DC, Library:Barrel_Jack, symbol Connector:Jack-DC
- added P1: USB_C_Plug_USB2.0, Connector_USB:USB_C_Receptacle_HRO_TYPE-C-31-M-12, symbol Connector:USB_C_Plug_USB2.0
- added Q1: FQPF8N60C, Package_TO_SOT_THT:TO-220F-3_Horizontal_TabDown, symbol Device:Q_NMOS_GDS
- added R1, R2: 100K, Resistor_THT:R_Axial_DIN0207_L6.3mm_D2.5mm_P7.62mm_Horizontal, symbol nigh_Library:R
- added SW1, SW2, SW3: SW_DIP_x01, Library:PWR_Switch_Pad, symbol Switch:SW_DIP_x01
- J13, J14, J16: renamed from J?; footprint (none) -> Library:Barrel_Jack
- J2, J3, J5, J6, J7, J8: renamed from J?; footprint (none) -> Connector_USB:USB_A_Molex_67643_Horizontal
Connections:
- net 5V is gone; now on net +5V: J2.1 (VBUS), J5.1 (VBUS), J7.1 (VBUS)
- net 5VSB: now also R2.1
- net GND: now also J1.15 (GND), J1.17 (GND), J1.18 (GND), J1.19 (GND), J1.24 (GND), J1.3 (GND), J1.5 (GND), J1.7 (GND), J13.2, J14.2, J16.2, J10.2 (Pin_2), J12.1 (Pin_1), J15.4 (Pin_4), J15.8 (Pin_8), J17.2 (Pin_2), J18.2 (Pin_2), J18.3 (Pin_3), J19.2 (Pin_2), J19.3 (Pin_3), J4.1 (Pin_1), J9.2, P1.A1 (GND), P1.A12 (GND), P1.B1 (GND), P1.B12 (GND), Q1.3 (S), R1.1, SW1.2
- net 12VO: now reaches J13.1
- net 12VO: now also J16.1, J10.1 (Pin_1), J17.1 (Pin_1), SW2.2, SW3.1
- net +3V3: now reaches J1.1 (+3.3V), J1.12 (+3.3V), J1.13 (+3.3V), J1.2 (+3.3V)
- net +12V: now reaches J1.10 (+12V), J1.11 (+12V)
- net +12V: now also J11.1 (Pin_1), J18.1 (Pin_1), J19.1 (Pin_1), SW2.1
- net -12V: now reaches J1.14 (-12V)
- net PS_ON: now reaches J1.16 (PS_ON#)
- net PS_ON: now also SW1.1
- net +5V: now reaches J1.21 (+5V), J1.22 (+5V), J1.23 (+5V), J1.4 (+5V), J1.6 (+5V)
- net +5V: now also J15.1 (Pin_1), J15.5 (Pin_5), J18.4 (Pin_4), J19.4 (Pin_4), J4.2 (Pin_2), P1.A4 (VBUS), P1.A9 (VBUS), P1.B4 (VBUS), P1.B9 (VBUS)
- net PWR_OK: now reaches J1.8 (PWR_OK)
- net PWR_OK: now also Q1.1 (G), R1.2
- net +5VP: now reaches J1.9 (+5VSB)
- net BAT1+: now reaches J14.1
- net BAT1+: now also J9.1, SW3.2
- new net: J12.2 (Pin_2), R2.2
- new net LED_GND: J11.2 (Pin_2), J11.3 (Pin_3), Q1.2 (D)
- new net PWR_SWITCH_N: J4.3 (Pin_3)
- new net PWR_SWITCH_P: J4.4 (Pin_4)
Other:
- moved on the sheet: H2, H4, H6, J1, J13, J14, J16, J2, J3, J5, J6, J7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
